File: _KiCad/MOSHield/MOSHield/MOSHield.kicad_pcb (KiCad board)
At the start: 2 copper layers, 68.6 x 53.3 mm, 8 parts, among them J1 Power, J2 Digital/PWM, J3 Analog, J4 Digital/PWM

Commit message: Added datasheet
Parts:
- added C1: 100n, Capacitor_THT:C_Disc_D4.7mm_W2.5mm_P5.00mm, F.Cu at (114.0, 86.1)
- added C2: 100n, Capacitor_THT:C_Disc_D4.7mm_W2.5mm_P5.00mm, F.Cu at (158.4, 91.1)
- added C3: 100n, Capacitor_THT:C_Disc_D4.7mm_W2.5mm_P5.00mm, F.Cu at (141.9, 83.5)
- added C4: 1u, Capacitor_THT:C_Rect_L7.0mm_W4.5mm_P5.00mm, F.Cu at (153.3, 81.0)
- added C5: 100n, Capacitor_THT:C_Disc_D4.7mm_W2.5mm_P5.00mm, F.Cu at (145.7, 101.3)
- added GS1: ~, Package_TO_SOT_THT:TO-5-10, F.Cu at (138.1, 63.2)
- added J5: Jumper, Connector_PinHeader_2.54mm:PinHeader_1x03_P2.54mm_Vertical, F.Cu at (144.4, 72.1)
- added J7: Conn_01x08, Connector_PinSocket_2.54mm:PinSocket_1x08_P2.54mm_Vertical, F.Cu at (105.6, 61.7)
- added Q1: IRF540N, Package_TO_SOT_THT:TO-220-3_Vertical, F.Cu at (153.7, 61.3)
- added R1: 100k, Resistor_THT:R_Axial_DIN0207_L6.3mm_D2.5mm_P10.16mm_Horizontal, F.Cu at (121.6, 81.0)
- added R3: 100k, Resistor_THT:R_Axial_DIN0207_L6.3mm_D2.5mm_P10.16mm_Horizontal, F.Cu at (147.0, 78.4)
- added R4: 1k, Resistor_THT:R_Axial_DIN0207_L6.3mm_D2.5mm_P10.16mm_Horizontal, F.Cu at (138.1, 81.0)
- added R5: 10k, Resistor_THT:R_Axial_DIN0207_L6.3mm_D2.5mm_P10.16mm_Horizontal, F.Cu at (114.0, 68.2)
- added R6: 1k, Resistor_THT:R_Axial_DIN0207_L6.3mm_D2.5mm_P10.16mm_Horizontal, F.Cu at (162.2, 78.4)
- added R7: 1k, Resistor_THT:R_Axial_DIN0207_L6.3mm_D2.5mm_P10.16mm_Horizontal, F.Cu at (153.3, 55.5)
- added R8: 10k, Resistor_THT:R_Axial_DIN0207_L6.3mm_D2.5mm_P10.16mm_Horizontal, F.Cu at (161.0, 69.5)
- added U1: LTC1050, Package_DIP:DIP-8_W7.62mm, F.Cu at (128.0, 81.0)
- added U2: MCP41100, Package_DIP:DIP-8_W7.62mm, F.Cu at (121.6, 59.4)
Connections:
- J1 pad 4: +3V3 -> unconnected-(J1-Pin_4-Pad4)
- J2 pad 5: /13 -> SCK
- J2 pad 7: /*11 -> SMOSI
- J2 pad 8: /*10 -> CS
- J3 pad 1: /A0 -> VADC_GAS
- J3 pad 2: /A1 -> VADC_TEMP
- J4 pad 2: /*6 -> RST
- J4 pad 3: /*5 -> RX
- J4 pad 4: /4 -> TX
- J4 pad 5: /*3 -> PWM
Routing:
- net +5V: track 0.00 -> 143.4 mm
- net TX: track 0.00 -> 68.4 mm
- net RST: track 0.00 -> 66.5 mm
- net RX: track 0.00 -> 64.8 mm
- net VCC: track 0.00 -> 59.4 mm
- net VADC_TEMP: track 0.00 -> 51.3 mm, vias 0 -> 2
- net R2: track 0.00 -> 48.2 mm, vias 0 -> 2
- net Net-(C4-Pad2): track 0.00 -> 46.9 mm, vias 0 -> 2
- net Net-(J5-Pin_2): track 0.00 -> 37.6 mm
- net VHEAT: track 0.00 -> 35.9 mm
- net SMOSI: track 0.00 -> 32.2 mm, vias 0 -> 2
- net Net-(U1-+): track 0.00 -> 26.3 mm
- net SCK: track 0.00 -> 22.4 mm
- net CS: track 0.00 -> 20.8 mm
- net IGAS2: track 0.00 -> 19.7 mm, vias 0 -> 2
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- added copper zone on B.Cu, net GND
Other:
- board size 68.6 x 53.3 mm -> 68.6 x 64.8 mm
