File: _KiCad/MOSHield2/MOSHield2/MOSHield2.kicad_pcb (KiCad board)
At the start: 2 copper layers, 69.8 x 61 mm, 23 parts, among them J1 Power, J2 Digital/PWM, J3 Analog, J4 Digital/PWM, J5 Jumper, J7 Conn_01x08, Q1 IRF540N, U1 LTC1050, U2 MCP41100

Commit message: Almost final commit
Routing:
- net GND: track 3.09 -> 7.58 mm, vias 0 -> 2
Changed lines of the file:
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@@
   (gr_line (start 100 44.12) (end 169.85 44.12)
     (stroke (width 0.15) (type solid)) (layer "Edge.Cuts"))
+  (segment (start 112.065 58.09) (end 115.24 61.265) (width 0.8) (layer "F.Cu") (net 1))
+  (via (at 115.24 61.265) (size 0.6) (drill 0.4) (layers "F.Cu" "B.Cu") (net 1))
+  (via (at 112.065 58.09) (size 0.6) (drill 0.4) (layers "F.Cu" "B.Cu") (free) (net 1))
   (segment (start 150.78 87.34) (end 152.08 86.04) (width 1.2) (layer "B.Cu") (net 1))
   (segment (start 150.78 87.34) (end 149.53 87.34) (width 1.2) (layer "B.Cu") (net 1))
